Commit message: Lab steps followed,  Could not contact service /controller_manager/list_controllers

File: src/ur3_description/urdf/ur3.gazebo.xacro (robot description, xacro)
@@ -1,6 +1,51 @@
 <?xml version="1.0"?>
 <robot xmlns:xacro="http://ros.org/wiki/xacro">
-  <gazebo>
-    <!-- add plugin info here -->
-  </gazebo>
+  <!-- ros_control plugin -->
+    <gazebo>
+        <plugin filename="gz_ros2_control-system" name="gz_ros2_control::GazeboSimROS2ControlPlugin">
+            <parameters>$(find ur3_description)/config/rrbot_controllers.yaml</parameters>
+        </plugin>
+    </gazebo>
+  <xacro:macro name="ur3_gazebo">
+    <!-- Base Link -->
+    <gazebo reference="base_link">
+      <material>Gazebo/Gray</material>
+    </gazebo>
+    <!-- Shoulder Link -->
+    <gazebo reference="shoulder_link">
+      <mu1>0.2</mu1>
+      <mu2>0.2</mu2>
+      <material>Gazebo/Blue</material>
+    </gazebo>
+    <!-- Upper Arm Link -->
+    <gazebo reference="upper_arm_link">
+      <mu1>0.2</mu1>
+      <mu2>0.2</mu2>
+      <material>Gazebo/Green</material>
+    </gazebo>
+    <!-- Forearm Link -->
+    <gazebo reference="forearm_link">
+      <mu1>0.2</mu1>
+      <mu2>0.2</mu2>
+      <material>Gazebo/Red</material>
+    </gazebo>
+    <!-- Wrist 1 Link -->
+    <gazebo reference="wrist_1_link">
+      <mu1>0.2</mu1>
+      <mu2>0.2</mu2>
+      <material>Gazebo/Yellow</material>
+    </gazebo>
+    <!-- Wrist 2 Link -->
+    <gazebo reference="wrist_2_link">
+      <mu1>0.2</mu1>
+      <mu2>0.2</mu2>
+      <material>Gazebo/Orange</material>
+    </gazebo>
+    <!-- Wrist 3 Link -->
+    <gazebo reference="wrist_3_link">
+      <mu1>0.2</mu1>
+      <mu2>0.2</mu2>
+      <material>Gazebo/Purple</material>
+    </gazebo>
+  </xacro:macro>
 </robot>

File: src/ur3_description/urdf/ur3.ros2_control.xacro (robot description, xacro)
@@ -3,5 +3,42 @@
   <xacro:macro name="ur3_ros2_control" params="name prefix">
     <ros2_control name="${name}" type="system">
-      <!-- add controller info here -->
+      <hardware>
+        <plugin>gz_ros2_control/GazeboSimSystem</plugin>
+      </hardware>
+      <joint name="${prefix}shoulder_lift_joint">
+          <command_interface name="position">
+              <param name="min">-1</param>
+              <param name="max">1</param>
+          </command_interface>
+          <state_interface name="position"/>
+      </joint>
+      <joint name="${prefix}elbow_joint">
+          <command_interface name="position">
+              <param name="min">-1</param>
+              <param name="max">1</param>
+          </command_interface>
+          <state_interface name="position"/>
+      </joint>
+      <joint name="${prefix}wrist_1_joint">
+          <command_interface name="position">
+              <param name="min">-1</param>
+              <param name="max">1</param>
+          </command_interface>
+          <state_interface name="position"/>
+      </joint>
+      <joint name="${prefix}wrist_2_joint">
+          <command_interface name="position">
+              <param name="min">-1</param>
+              <param name="max">1</param>
+          </command_interface>
+          <state_interface name="position"/>
+      </joint>
+      <joint name="${prefix}wrist_3_joint">
+          <command_interface name="position">
+              <param name="min">-1</param>
+              <param name="max">1</param>
+          </command_interface>
+          <state_interface name="position"/>
+      </joint>
     </ros2_control>
   </xacro:macro>

File: src/ur3_description/urdf/ur3.urdf.xacro (robot description, xacro)
@@ -59,7 +59,9 @@
      <origin xyz="0 0 0" rpy="0 0 0" />          <!-- position robot in the world -->
    </xacro:ur_robot>
-   <!-- call ur3 ros2_control macro -->
+   <!-- call ur3_ros2_control macro -->
+   <xacro:include filename="$(find ur3_description)/urdf/ur3.ros2_control.xacro" />
    <xacro:ur3_ros2_control name="$(arg name)" prefix="$(arg prefix)"/>
    <!-- gazebo classic plugin -->
    <xacro:include filename="$(find ur3_description)/urdf/ur3.gazebo.xacro" />
+   <xacro:ur3_gazebo/>
 </robot>
