Commit message: shoulder pan

File: src/ur3_description/urdf/ur3.ros2_control.xacro (robot description, xacro)
@@ -6,4 +6,11 @@
         <plugin>gz_ros2_control/GazeboSimSystem</plugin>
       </hardware>
+      <joint name="${prefix}shoulder_pan_joint">
+         <command_interface name="position">
+             <param name="min">-6.28</param>
+             <param name="max">6.28</param>
+         </command_interface>
+         <state_interface name="position"/>
+      </joint>
       <joint name="${prefix}shoulder_lift_joint">
           <command_interface name="position">
